File: Adaptateurs_NiveauxSPI/Adaptateurs_NiveauxSPI.sch (KiCad schematic (older format))
At the start: 21 parts, among them P1 CONN_01X07, P2 CONN_01X08, P3 CONN_01X07, P4 CONN_01X12, P5 CONN_01X07, P6 CONN_01X09, P7 CONN_01X07, P8 CONN_01X10, U1 CON_5V_3-3V, U2 CON_5V_3-3V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

Commit message: Update projet
- Add RFM95W
- Add MPM 4in1
Parts:
- added C10, C11, C12, C9: 100nF, Capacitor_SMD:C_1206_3216Metric_Pad1.42x1.75mm_HandSolder, symbol Adaptateurs_NiveauxSPI-rescue:C-device
- added J1: RFM95W, Conv_SPI:RFM95W, symbol Connector_Generic:Conn_01x16
- added J2: MPM_ 4en1, Connector_PinHeader_2.00mm:PinHeader_2x05_P2.00mm_Vertical, symbol Connector_Generic:Conn_01x10
- added J3: MPM_4in1, Connector_PinHeader_2.54mm:PinHeader_1x03_P2.54mm_Vertical, symbol Connector_Generic:Conn_01x03
- added J4: SMA, Conv_SPI:SMA_Amphenol_132289_EdgeMount, symbol Connector_Generic:Conn_01x02
- added P10: SpirfMod, Connector_PinHeader_2.54mm:PinHeader_2x05_P2.54mm_Vertical, symbol Connector_Generic:Conn_01x10
- added P9: SpirfMod, Connector_PinHeader_2.54mm:PinHeader_1x07_P2.54mm_Vertical, symbol Mega_2560-core-mini_full_2.1:CONN_01X07
- added U5: CONV_5V/3.3V, Conv_SPI:Level_Convertissor_SMD, symbol Adaptateurs_NiveauxSPI-rescue:CON_5V_3-3V
- added U6: CONV_5V_3-3V_8, Conv_SPI:Level_Convertissor_8_W10.16mm, symbol Adaptateurs_NiveauxSPI-rescue:CONV_5V_3-3V_8
- C1, C2, C3, C4, C5, C6, C7, C8: footprint C_1206 -> Capacitor_SMD:C_1206_3216Metric_Pad1.42x1.75mm_HandSolder; symbol C -> Adaptateurs_NiveauxSPI-rescue:C-device
- P1, P3: value CONN_01X07 -> SpirfMod; footprint Pin_Header_Straight_1x07_Pitch2.54mm -> Connector_PinHeader_2.54mm:PinHeader_1x07_P2.54mm_Vertical; symbol CONN_01X07 -> Mega_2560-core-mini_full_2.1:CONN_01X07
- P2: value CONN_01X08 -> NRF24L01; footprint Pin_Header_Straight_2x04_Pitch2.54mm -> Connector_PinHeader_2.54mm:PinHeader_2x04_P2.54mm_Vertical; symbol CONN_01X08 -> Mega_2560-core-mini_full_2.1:CONN_01X08
- P4: value CONN_01X12 -> CC2500; footprint Pin_Header_Straight_2x06_Pitch2.54mm -> Connector_PinHeader_2.54mm:PinHeader_2x06_P2.54mm_Vertical; symbol CONN_01X12 -> Mega_2560-core-mini_full_2.1:CONN_01X12
- P5: value CONN_01X07 -> SpirMod; footprint Pin_Header_Straight_1x07_Pitch2.54mm -> Connector_PinHeader_2.54mm:PinHeader_1x07_P2.54mm_Vertical; symbol CONN_01X07 -> Mega_2560-core-mini_full_2.1:CONN_01X07
- P6: value CONN_01X09 -> A7105; footprint Pin_Header_Straight_1x09_Pitch2.54mm -> Conv_SPI:Pin_Header_Straight_1x09_Pitch2mm; symbol CONN_01X09 -> Mega_2560-core-mini_full_2.1:CONN_01X09
- P7: footprint Pin_Header_Straight_1x07_Pitch2.54mm -> Connector_PinHeader_2.54mm:PinHeader_1x07_P2.54mm_Vertical; symbol CONN_01X07 -> Mega_2560-core-mini_full_2.1:CONN_01X07
- P8: footprint Pin_Header_Straight_2x05_Pitch2.54mm -> Connector_PinHeader_2.54mm:PinHeader_2x05_P2.54mm_Vertical; symbol CONN_01X10 -> Mega_2560-core-mini_full_2.1:CONN_01X10
- R1: footprint R_1206 -> Resistor_SMD:R_1206_3216Metric_Pad1.42x1.75mm_HandSolder; symbol R -> Adaptateurs_NiveauxSPI-rescue:R-device
- U1, U2, U3, U4: value CON_5V_3-3V -> CONV_5V/3.3V; symbol CON_5V_3-3V -> Adaptateurs_NiveauxSPI-rescue:CON_5V_3-3V
Connections:
- net labels added: +3.3VA, +5F, +5VL, 24L01, A7105, CC2500, CS-CC2500, CS_A7105, CS_CYRF, CS_NRF24L01, CYRF, GNDREF, GNDS, MISO, MISO_L, MOSI, MOSI_L, SCK, SCK_L
- wire segments 148 -> 260
Other:
- note added: "Adaptateur 5v/3,3v SPI pour le MPM 4 en 1"
- note added: "Adaptateur 5v/3,3v SPI pour le RFM95W"
- note added: "CS_CYRF"
- note added: "MISO"
- note added: "MOSI"
- note added: "NSS"
- note added: "SCK"
- moved on the sheet: U1, U2, U3, U4
